File: eagle/EFM_VCF3.brd (EAGLE design)
At the start: 100 x 80.6 mm, 21 parts, among them IC1 LM13700N, Q3 2N3906, Q4 2N3906, U1 POWER

Commit message: started the board
Parts:
- removed CV1, CV1_NORM, CV2: LSP10, solpad:LSP10
- removed CV2_LEVEL: 100k, pot:3RP/1610N
- added BP_OUT, CV_1, HP_OUT, IN_1, LP_OUT: AUDIO-JACK, erthenvar:ERTHENVAR-JACK-90DEG
- added C3, C4: 220p, rcl:C075-032X103
- added CV1_LEVEL, IN1_LEV: 100k, pot:3RP/1610N
- added IC2: TL084P, linear:DIL14
- added Q: 50k, pot:3RP/1610N
- added R10, R13, R14, R15, R16, R17, R9: 1k, rcl:0207/7
- added R18, R19, R20, R21, R5: 100k, rcl:0207/7
- added R22: 10k, rcl:0207/7
- added SCALE_TRIM: 10k, rcl:RTRIM64W
- R7: value 100k -> 10k
- moved R4 101.6 mm to (68.6, 45.7), turned to 90 degrees
- moved R3 93.3 mm to (61.0, 45.7), turned to 270 degrees
- moved R2 75.5 mm to (63.5, 22.9), turned to 180 degrees
- moved U1 74.5 mm to (11.4, 50.8)
- moved R1 69.9 mm to (63.5, 17.8), turned to 180 degrees
- moved Q4 50.3 mm to (38.1, 20.3)
- moved R12 32.7 mm to (48.3, 25.4), turned to 0 degrees
- moved R7 28.1 mm to (33.0, 36.8), turned to 180 degrees
- moved Q3 27.4 mm to (45.7, 20.3), turned to 90 degrees
- moved C2 23.1 mm to (20.3, 55.9)
- moved IC1 15.5 mm to (48.3, 45.7), turned to 0 degrees
- moved C1 12.9 mm to (20.3, 48.3), turned to 90 degrees
- moved CUTOFF_INIT 11.7 mm to (30.5, 33.0), turned to 270 degrees
- moved R11 9.67 mm to (34.3, 27.9), turned to 180 degrees
- moved CUTOFF 4.62 mm to (80.0, 3.81)
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Connections:
- removed net N$53: R7.2
- removed net N$59: CV1.MP
- new net N$11: IC2.5, R15.2
- new net N$12: IC2.10, R16.2
- new net N$13: IC2.12, R17.2
- new net N$14: IC2.13, IC2.14, LP_OUT.P$3
- new net N$15: BP_OUT.P$3, IC2.8, IC2.9
- new net N$17: HP_OUT.P$3, IC2.6, IC2.7
- new net N$18: Q3.2, R11.1, R12.1, R6.1, R8.1
- new net N$19: Q.2, R18.2
- new net N$2: C3.1, IC1.10, IC1.12
- new net N$20: IC1.16, R22.1
- new net N$21: R22.2, R7.2, SCALE_TRIM.3
- new net N$22: IN1_LEV.3, IN_1.P$3
- new net N$23: IC1.8, R17.1, R19.2, R4.1
- new net N$24: IN1_LEV.2, R21.1
- new net N$25: Q4.1, SCALE_TRIM.1, SCALE_TRIM.2
- new net N$26: IC2.2, R18.1, R19.1, R20.1, R21.2
- new net N$3: C4.1, IC1.5, IC1.7
- new net N$4: IC1.14, R5.2, R9.1
- new net N$5: IC1.9, Q.3, R16.1, R2.1, R3.1
- new net N$6: IC1.3, R14.1, R2.2
- new net N$7: IC1.13, R10.1
- new net N$8: IC1.4, R13.1
- new net N$9: IC2.1, R15.1, R20.2, R5.1
- net +12V: now also IC2.4
- net -12V: now also CUTOFF.1, IC2.11, R3.2, R4.2
- net GND: now also BP_OUT.P$1, C3.2, C4.2, CV1_LEVEL.1, CV_1.P$1, HP_OUT.P$1, IC2.3, IN1_LEV.1, IN_1.P$1, LP_OUT.P$1, Q.1, R10.2, R13.2, R14.2, R9.2; no longer CUTOFF.1, CV2_LEVEL.1
- net N$10: now also CV1_LEVEL.2; no longer CV2_LEVEL.2
- net N$16: now also IC1.1; no longer Q3.2, R11.1, R12.1, R6.1, R8.1
- net N$54: now also CV1_LEVEL.3, CV_1.P$3; no longer CV2.MP, CV2_LEVEL.3
- net N$55: now also CV_1.P$2; no longer CV1_NORM.MP
Routing:
- net -12V: track 41.6 -> 258.0 mm, vias 2 -> 0
- net N$5: track 0.00 -> 160.8 mm
- net N$16: track 90.4 -> 6.13 mm, vias 2 -> 0
- net N$26: track 0.00 -> 83.5 mm
- net N$4: track 0.00 -> 82.2 mm
- net N$18: track 0.00 -> 74.8 mm
- net GND: track 280.1 -> 220.8 mm, vias 2 -> 0
- net N$23: track 0.00 -> 58.8 mm
- net N$1: track 0.00 -> 52.0 mm
- net N$19: track 0.00 -> 50.7 mm
- net N$6: track 0.00 -> 29.1 mm
- net N$9: track 0.00 -> 26.7 mm
- net N$38: track 83.6 -> 62.5 mm
- net N$27: track 32.6 -> 12.0 mm
- net N$25: track 0.00 -> 18.6 mm
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Other:
- board size 100 x 80.6 mm -> 100 x 80 mm

Commit message: working on brd
Parts:
- added BP_GND, HP_GND: LSP10, solpad:LSP10
- BP_OUT, HP_OUT: value AUDIO-JACK -> LSP10; device erthenvar:ERTHENVAR-JACK-90DEG -> solpad:LSP10
- moved CUTOFF_INIT 53.9 mm to (82.5, 19.1), turned to 90 degrees
- moved R11 44.6 mm to (78.7, 24.1), turned to 0 degrees
- moved BP_OUT 44.6 mm to (73.7, 38.1), turned to 0 degrees
- moved HP_OUT 27.1 mm to (74.9, 53.3), turned to 0 degrees
- moved R21 9.67 mm to (57.1, 67.3), turned to 270 degrees
Connections:
- net GND: now also BP_GND.MP, HP_GND.MP; no longer BP_OUT.P$1, HP_OUT.P$1
- net N$15: now also BP_OUT.MP; no longer BP_OUT.P$3
- net N$17: now also HP_OUT.MP; no longer HP_OUT.P$3
Routing:
- net -12V: track 258.0 -> 0.00 mm
- net GND: track 220.8 -> 0.00 mm
- net N$5: track 160.8 -> 0.00 mm
- net N$26: track 83.5 -> 0.00 mm
- net N$4: track 82.2 -> 0.00 mm
- net N$18: track 74.8 -> 0.00 mm
- net N$38: track 62.5 -> 0.00 mm
- net N$23: track 58.8 -> 0.00 mm
- net N$1: track 52.0 -> 0.00 mm
- net N$19: track 50.7 -> 0.00 mm
- net N$6: track 29.1 -> 0.00 mm
- net N$9: track 26.7 -> 0.00 mm
- net N$25: track 18.6 -> 0.00 mm
- net N$21: track 18.4 -> 0.00 mm
- net N$27: track 12.0 -> 0.00 mm
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
Commit message: almost routed
Parts:
- moved R18 16.6 mm to (63.5, 29.2)
- moved HP_GND 10.2 mm to (62.2, 57.1)
- moved R12 7.73 mm to (55.9, 24.1), turned to 90 degrees
- moved SCALE_TRIM 7.41 mm to (30.5, 27.9)
- moved R19 6.35 mm to (67.3, 35.6)
- moved R16 5.68 mm to (81.3, 30.5), turned to 180 degrees
- moved BP_GND 5.24 mm to (63.5, 53.3)
- moved R17 5.24 mm to (78.7, 34.3), turned to 0 degrees
- moved Q4 4.02 mm to (36.8, 24.1), turned to 270 degrees
- moved R9 3.81 mm to (40.6, 64.8)
- moved R6 2.84 mm to (71.1, 11.4)
- moved C3 2.54 mm to (52.1, 61.0)
- moved Q3 2.54 mm to (45.7, 22.9), turned to 180 degrees
- moved R15 2.54 mm to (78.7, 58.4)
- moved R10 1.80 mm to (47.0, 59.7)
Routing:
- net GND: track 0.00 -> 414.7 mm
- net N$38: track 0.00 -> 164.5 mm
- net N$5: track 0.00 -> 157.4 mm
- net -12V: track 0.00 -> 140.5 mm
- net N$24: track 0.00 -> 129.1 mm
- net N$26: track 0.00 -> 80.6 mm
- net N$18: track 0.00 -> 55.6 mm
- net N$4: track 0.00 -> 53.7 mm
- net N$23: track 0.00 -> 42.2 mm
- net N$1: track 0.00 -> 40.8 mm
- net +12V: track 0.00 -> 36.8 mm, vias 0 -> 2
- net N$9: track 0.00 -> 33.6 mm
- net N$6: track 0.00 -> 29.8 mm
- net N$22: track 0.00 -> 28.1 mm
- net N$2: track 0.00 -> 18.6 mm
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
Commit message: gcode
Parts:
- moved R11 15.5 mm to (66.0, 15.2)
- moved R8 6.48 mm to (52.1, 11.4)
- moved R9 6.35 mm to (44.5, 59.7), turned to 90 degrees
- moved R6 5.08 mm to (66.0, 11.4)
- moved BP_GND 4.58 mm to (59.7, 55.9)
- moved CUTOFF_INIT 4.02 mm to (78.7, 20.3), turned to 0 degrees
- moved R21 3.18 mm to (59.1, 64.8)
- moved R1 2.84 mm to (66.0, 19.1)
- moved R18 2.54 mm to (63.5, 31.8)
- moved R19 2.54 mm to (67.3, 38.1)
- moved R2 2.54 mm to (63.5, 25.4)
- moved R7 2.54 mm to (35.6, 36.8)
- moved HP_GND 1.80 mm to (63.5, 55.9)
- moved Q3 1.80 mm to (44.5, 24.1)
- moved R22 1.42 mm to (33.0, 45.1)
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Routing:
- net GND: track 414.7 -> 511.2 mm
- net N$55: track 2.54 -> 56.1 mm, vias 0 -> 2
- net N$54: track 0.00 -> 31.5 mm
- net N$14: track 2.54 -> 30.9 mm, vias 0 -> 2
- net N$19: track 0.00 -> 26.2 mm
- net N$4: track 53.7 -> 29.9 mm
- net N$5: track 157.4 -> 133.8 mm
- net N$38: track 164.5 -> 143.7 mm
- net N$18: track 55.6 -> 40.5 mm
- net -12V: track 140.5 -> 153.5 mm, vias 0 -> 2
- net N$27: track 3.81 -> 11.4 mm
- net N$56: track 12.7 -> 18.8 mm
- net N$26: track 80.6 -> 75.5 mm
- net N$10: track 12.0 -> 7.75 mm
- net N$6: track 29.8 -> 26.7 mm
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Other:
- board size 100 x 80 mm -> 102.2 x 80.6 mm

Commit message: fixed connections
Parts:
- R22: device rcl:0207/7 -> rcl:0309/10
- moved R12 5.24 mm to (57.1, 19.1)
- moved HP_GND 2.54 mm to (66.0, 55.9)
- moved R9 2.54 mm to (41.9, 59.7)
- moved BP_GND 2.54 mm to (62.2, 55.9)
- moved R17 1.27 mm to (80.0, 34.3)
- moved R10 1.27 mm to (45.7, 59.7)
- moved R11 1.27 mm to (66.0, 16.5)
- moved R1 1.27 mm to (66.0, 20.3)
- moved R16 1.27 mm to (82.5, 30.5)
- moved R22 1.27 mm to (34.3, 45.1)
Connections:
- removed net N$38: C1.+, CUTOFF.3, CUTOFF_INIT.3, R1.1, U1.10, U1.9
- net +12V: now also C1.+, CUTOFF.3, CUTOFF_INIT.3, R1.1, U1.10, U1.9
Routing:
- net +12V: track 35.6 -> 224.8 mm, vias 2 -> 4
- net N$38: track 143.7 -> 0.00 mm
- net -12V: track 153.5 -> 163.6 mm
- net N$18: track 40.5 -> 34.3 mm
- net N$4: track 29.9 -> 35.1 mm
- net N$56: track 18.8 -> 14.7 mm
- net N$2: track 17.6 -> 21.2 mm
- net N$55: track 56.1 -> 52.7 mm
- net GND: track 511.2 -> 513.9 mm
- net N$23: track 40.3 -> 42.5 mm
- net N$19: track 26.2 -> 24.3 mm
- net N$1: track 42.7 -> 41.4 mm
- net N$20: track 6.38 -> 5.12 mm
- net N$14: track 30.9 -> 29.9 mm
- net N$21: track 11.0 -> 10.4 mm

Commit message: tweaked
Parts:
- moved R12 2.84 mm to (55.9, 21.6)
- moved C4 1.80 mm to (53.3, 34.3)
- moved R1 1.27 mm to (66.0, 21.6)
- moved R11 1.27 mm to (66.0, 17.8)
Routing:
- net GND: track 513.9 -> 519.1 mm
- net N$24: track 129.8 -> 126.4 mm
- net N$3: track 11.8 -> 9.72 mm
- net N$18: track 34.3 -> 36.1 mm
- net N$27: track 11.7 -> 10.9 mm
