File: eagle/EFM_VCF3.sch (EAGLE design)
At the start: 21 parts, among them IC1 LM13700N, Q3 2N3906, Q4 2N3906, U1 POWER

Commit message: more parts
Parts:
- added C3, C4: 220p, rcl:C-US075-032X103
- added R10, R13, R14, R15, R16, R17, R9: 1k, rcl:R-US_0207/7
- added R5: 100k, rcl:R-US_0207/7
Connections:
- new net N$2: C3.1, IC1B.OUT, IC1G$4.IN
- new net N$3: C4.1, IC1A.OUT, IC1G$3.IN
- new net N$4: IC1B.+IN, R5.2, R9.1
- new net N$5: IC1G$4.OUT, R2.1, R3.1
- new net N$6: IC1A.+IN, R14.1, R2.2
- new net N$7: IC1B.-IN, R10.1
- new net N$8: IC1A.-IN, R13.1
- net -12V: now also R3.2, R4.2
- net GND: now also C3.2, C4.2, R10.2, R13.2, R14.2, R9.2
Other:
- moved on the sheet: R3, R4
Changed lines of the file:
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@@
 <part name="R3" library="rcl" deviceset="R-US_" device="0207/7" value="10k"/>
 <part name="R4" library="rcl" deviceset="R-US_" device="0207/7" value="10k"/>
+<part name="C3" library="rcl" deviceset="C-US" device="075-032X103" value="220p"/>
+<part name="C4" library="rcl" deviceset="C-US" device="075-032X103" value="220p"/>
+<part name="GND3" library="supply1" deviceset="GND" device=""/>
+<part name="GND6" library="supply1" deviceset="GND" device=""/>
+<part name="P-5" library="supply1" deviceset="-12V" device=""/>
+<part name="P-6" library="supply1" deviceset="-12V" device=""/>
+<part name="R5" library="rcl" deviceset="R-US_" device="0207/7" value="100k"/>
+<part name="R9" library="rcl" deviceset="R-US_" device="0207/7" value="1k"/>
+<part name="R10" library="rcl" deviceset="R-US_" device="0207/7" value="1k"/>
+<part name="R13" library="rcl" deviceset="R-US_" device="0207/7" value="1k"/>
+<part name="R14" library="rcl" deviceset="R-US_" device="0207/7" value="1k"/>
+<part name="GND7" library="supply1" deviceset="GND" device=""/>
+<part name="GND8" library="supply1" deviceset="GND" device=""/>
+<part name="GND11" library="supply1" deviceset="GND" device=""/>
+<part name="GND12" library="supply1" deviceset="GND" device=""/>
+<part name="R15" library="rcl" deviceset="R-US_" device="0207/7" value="1k"/>
+<part name="R16" library="rcl" deviceset="R-US_" device="0207/7" value="1k"/>
+<part name="R17" library="rcl" deviceset="R-US_" device="0207/7" value="1k"/>
 </parts>
 <sheets>
@@
 <instances>
 <instance part="IC1" gate="A" x="86.36" y="109.22"/>
-<instance part="IC1" gate="G$3" x="83.82" y="134.62"/>
+<instance part="IC1" gate="G$3" x="119.38" y="109.22"/>
 <instance part="IC1" gate="G$4" x="27.94" y="104.14"/>
 <instance part="IC1" gate="B" x="-5.08" y="104.14"/>
@@
 <instance part="P+6" gate="1" x="-5.08" y="73.66"/>
 <instance part="R2" gate="G$1" x="55.88" y="104.14"/>
-<instance part="R3" gate="G$1" x="40.64" y="91.44" rot="R270"/>
-<instance part="R4" gate="G$1" x="119.38" y="91.44" rot="R270"/>
+<instance part="R3" gate="G$1" x="45.72" y="93.98" rot="R270"/>
+<instance part="R4" gate="G$1" x="132.08" y="99.06" rot="R270"/>
+<instance part="C3" gate="G$1" x="17.78" y="96.52"/>
+<instance part="C4" gate="G$1" x="109.22" y="101.6"/>
+<instance part="GND3" gate="1" x="17.78" y="86.36"/>
+<instance part="GND6" gate="1" x="109.22" y="91.44"/>
+<instance part="P-5" gate="1" x="45.72" y="83.82"/>
+<instance part="P-6" gate="1" x="132.08" y="88.9"/>
+<instance part="R5" gate="G$1" x="-30.48" y="99.06"/>
+<instance part="R9" gate="G$1" x="-22.86" y="91.44" rot="R270"/>
+<instance part="R10" gate="G$1" x="-17.78" y="91.44" rot="R270"/>
+<instance part="R13" gate="G$1" x="73.66" y="93.98" rot="R270"/>
+<instance part="R14" gate="G$1" x="68.58" y="93.98" rot="R270"/>
+<instance part="GND7" gate="1" x="68.58" y="86.36"/>
+<instance part="GND8" gate="1" x="73.66" y="86.36"/>
+<instance part="GND11" gate="1" x="-17.78" y="83.82"/>
+<instance part="GND12" gate="1" x="-22.86" y="83.82"/>
+<instance part="R15" gate="G$1" x="147.32" y="142.24"/>
+<instance part="R16" gate="G$1" x="147.32" y="127"/>
+<instance part="R17" gate="G$1" x="147.32" y="111.76"/>
 </instances>
 <busses>
@@
 <pinref part="GND9" gate="1" pin="GND"/>
 </segment>
+<segment>
+<pinref part="C3" gate="G$1" pin="2"/>
+<pinref part="GND3" gate="1" pin="GND"/>
+<wire x1="17.78" y1="91.44" x2="17.78" y2="88.9" width="0.1524" layer="91"/>
+</segment>
+<segment>
+<pinref part="C4" gate="G$1" pin="2"/>
+<pinref part="GND6" gate="1" pin="GND"/>
+<wire x1="109.22" y1="93.98" x2="109.22" y2="96.52" width="0.1524" layer="91"/>
+</segment>
+<segment>
+<pinref part="R14" gate="G$1" pin="2"/>
+<pinref part="GND7" gate="1" pin="GND"/>
+</segment>
+<segment>
+<pinref part="R13" gate="G$1" pin="2"/>
+<pinref part="GND8" gate="1" pin="GND"/>
+</segment>
+<segment>
+<pinref part="R10" gate="G$1" pin="2"/>
+<pinref part="GND11" gate="1" pin="GND"/>
+</segment>
+<segment>
+<pinref part="R9" gate="G$1" pin="2"/>
+<pinref part="GND12" gate="1" pin="GND"/>
+</segment>
 </net>
 <net name="N$38" class="0">
@@
 <wire x1="66.04" y1="27.94" x2="66.04" y2="24.384" width="0.1524" layer="91"/>
 <pinref part="C2" gate="G$1" pin="-"/>
+</segment>
+<segment>
+<pinref part="R3" gate="G$1" pin="2"/>
+<pinref part="P-5" gate="1" pin="-12V"/>
+<wire x1="45.72" y1="88.9" x2="45.72" y2="86.36" width="0.1524" layer="91"/>
+</segment>
+<segment>
+<pinref part="R4" gate="G$1" pin="2"/>
+<pinref part="P-6" gate="1" pin="-12V"/>
+<wire x1="132.08" y1="91.44" x2="132.08" y2="93.98" width="0.1524" layer="91"/>
 </segment>
 </net>
@@
 </segment>
 </net>
+<net name="N$2" class="0">
+<segment>
+<pinref part="IC1" gate="B" pin="OUT"/>
+<pinref part="IC1" gate="G$4" pin="IN"/>
+<wire x1="20.32" y1="104.14" x2="17.78" y2="104.14" width="0.1524" layer="91"/>
+<pinref part="C3" gate="G$1" pin="1"/>
+<wire x1="17.78" y1="104.14" x2="15.24" y2="104.14" width="0.1524" layer="91"/>
+<wire x1="17.78" y1="99.06" x2="17.78" y2="104.14" width="0.1524" layer="91"/>
+<junction x="17.78" y="104.14"/>
+</segment>
+</net>
+<net name="N$3" class="0">
+<segment>
+<pinref part="IC1" gate="A" pin="OUT"/>
+<pinref part="IC1" gate="G$3" pin="IN"/>
+<wire x1="111.76" y1="109.22" x2="109.22" y2="109.22" width="0.1524" layer="91"/>
+<pinref part="C4" gate="G$1" pin="1"/>
+<wire x1="109.22" y1="109.22" x2="106.68" y2="109.22" width="0.1524" layer="91"/>
+<wire x1="109.22" y1="104.14" x2="109.22" y2="109.22" width="0.1524" layer="91"/>
+<junction x="109.22" y="109.22"/>
+</segment>
+</net>
+<net name="N$4" class="0">
+<segment>
+<pinref part="IC1" gate="B" pin="+IN"/>
+<pinref part="R5" gate="G$1" pin="2"/>
+<wire x1="-25.4" y1="99.06" x2="-22.86" y2="99.06" width="0.1524" layer="91"/>
+<pinref part="R9" gate="G$1" pin="1"/>
+<wire x1="-22.86" y1="99.06" x2="-15.24" y2="99.06" width="0.1524" layer="91"/>
+<wire x1="-22.86" y1="96.52" x2="-22.86" y2="99.06" width="0.1524" layer="91"/>
+<junction x="-22.86" y="99.06"/>
+</segment>
+</net>
+<net name="N$5" class="0">
+<segment>
+<pinref part="IC1" gate="G$4" pin="OUT"/>
+<pinref part="R2" gate="G$1" pin="1"/>
+<wire x1="50.8" y1="104.14" x2="45.72" y2="104.14" width="0.1524" layer="91"/>
+<pinref part="R3" gate="G$1" pin="1"/>
+<wire x1="45.72" y1="104.14" x2="35.56" y2="104.14" width="0.1524" layer="91"/>
+<wire x1="45.72" y1="99.06" x2="45.72" y2="104.14" width="0.1524" layer="91"/>
+<junction x="45.72" y="104.14"/>
+</segment>
+</net>
+<net name="N$6" class="0">
+<segment>
+<pinref part="IC1" gate="A" pin="+IN"/>
+<pinref part="R2" gate="G$1" pin="2"/>
+<wire x1="60.96" y1="104.14" x2="68.58" y2="104.14" width="0.1524" layer="91"/>
+<pinref part="R14" gate="G$1" pin="1"/>
+<wire x1="68.58" y1="104.14" x2="76.2" y2="104.14" width="0.1524" layer="91"/>
+<wire x1="68.58" y1="99.06" x2="68.58" y2="104.14" width="0.1524" layer="91"/>
+<junction x="68.58" y="104.14"/>
+</segment>
+</net>
+<net name="N$7" class="0">
+<segment>
+<pinref part="R10" gate="G$1" pin="1"/>
+<wire x1="-17.78" y1="96.52" x2="-17.78" y2="109.22" width="0.1524" layer="91"/>
+<pinref part="IC1" gate="B" pin="-IN"/>
+<wire x1="-17.78" y1="109.22" x2="-15.24" y2="109.22" width="0.1524" layer="91"/>
+</segment>
+</net>
+<net name="N$8" class="0">
+<segment>
+<pinref part="IC1" gate="A" pin="-IN"/>
+<pinref part="R13" gate="G$1" pin="1"/>
+<wire x1="76.2" y1="114.3" x2="73.66" y2="114.3" width="0.1524" layer="91"/>
+<wire x1="73.66" y1="114.3" x2="73.66" y2="99.06" width="0.1524" layer="91"/>
+</segment>
+</net>

Commit message: more parts
Parts:
- added IC2: TL084P, linear:TL084P
- added U$1: AUDIO-JACK, erthenvar:AUDIO-JACK
Connections:
- new net N$11: IC2B.+IN, R15.2
- new net N$12: IC2C.+IN, R16.2
- new net N$13: IC2D.+IN, R17.2
- new net N$9: IC2A.OUT, R5.1
- net +12V: now also IC2P.V+
- net -12V: now also CUTOFF.A, IC2P.V-
- net GND: no longer CUTOFF.A
Other:
- moved on the sheet: C1, C2, R12, U1
Changed lines of the file:
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@@
 <part name="P+3" library="supply1" deviceset="+12V" device=""/>
 <part name="R6" library="rcl" deviceset="R-US_" device="0207/7" value="100k"/>
-<part name="GND2" library="supply1" deviceset="GND" device=""/>
 <part name="CV1" library="solpad" deviceset="LSP10" device=""/>
 <part name="CV1_NORM" library="solpad" deviceset="LSP10" device=""/>
@@
 <part name="R16" library="rcl" deviceset="R-US_" device="0207/7" value="1k"/>
 <part name="R17" library="rcl" deviceset="R-US_" device="0207/7" value="1k"/>
+<part name="P-7" library="supply1" deviceset="-12V" device=""/>
+<part name="IC2" library="linear" deviceset="TL084" device="P"/>
+<part name="P+7" library="supply1" deviceset="+12V" device=""/>
+<part name="P-8" library="supply1" deviceset="-12V" device=""/>
+<part name="U$1" library="erthenvar" deviceset="AUDIO-JACK" device=""/>
 </parts>
 <sheets>
@@
 <instance part="IC1" gate="G$4" x="27.94" y="104.14"/>
 <instance part="IC1" gate="B" x="-5.08" y="104.14"/>
-<instance part="U1" gate="G$1" x="-86.36" y="116.84"/>
-<instance part="P+2" gate="1" x="-73.66" y="129.54"/>
-<instance part="P-2" gate="1" x="-68.58" y="109.22"/>
-<instance part="GND5" gate="1" x="-63.5" y="116.84"/>
-<instance part="IC1" gate="G$5" x="48.26" y="30.48"/>
+<instance part="U1" gate="G$1" x="35.56" y="38.1"/>
+<instance part="P+2" gate="1" x="48.26" y="50.8"/>
+<instance part="P-2" gate="1" x="53.34" y="30.48"/>
+<instance part="GND5" gate="1" x="58.42" y="38.1"/>
+<instance part="IC1" gate="G$5" x="114.3" y="30.48"/>
 <instance part="CV2_LEVEL" gate="G$1" x="-71.12" y="17.78"/>
 <instance part="GND4" gate="1" x="-71.12" y="7.62"/>
@@
 <instance part="P-4" gate="1" x="-30.48" y="-10.16"/>
 <instance part="R7" gate="G$1" x="-55.88" y="45.72" rot="R180"/>
-<instance part="P+4" gate="1" x="40.64" y="60.452"/>
-<instance part="P-3" gate="1" x="40.64" y="14.224"/>
+<instance part="P+4" gate="1" x="106.68" y="60.452"/>
+<instance part="P-3" gate="1" x="106.68" y="14.224"/>
 <instance part="CUTOFF" gate="G$1" x="-73.66" y="68.58"/>
 <instance part="P+3" gate="1" x="-73.66" y="78.74"/>
 <instance part="R6" gate="G$1" x="-55.88" y="68.58" rot="R180"/>
-<instance part="GND2" gate="1" x="-73.66" y="58.42"/>
 <instance part="CV1" gate="1" x="-76.2" y="45.72" rot="R90"/>
 <instance part="CV1_NORM" gate="1" x="-86.36" y="45.72" rot="R270"/>
 <instance part="CV2" gate="1" x="-83.82" y="30.48" rot="R90"/>
-<instance part="P+1" gate="1" x="66.04" y="57.912"/>
-<instance part="P-1" gate="1" x="66.04" y="21.844"/>
-<instance part="GND1" gate="1" x="55.88" y="33.02"/>
+<instance part="P+1" gate="1" x="132.08" y="57.912"/>
+<instance part="P-1" gate="1" x="132.08" y="21.844"/>
+<instance part="GND1" gate="1" x="121.92" y="33.02"/>
 <instance part="R11" gate="G$1" x="-43.18" y="7.62" rot="R270"/>
-<instance part="C1" gate="G$1" x="66.04" y="48.26"/>
-<instance part="C2" gate="G$1" x="66.04" y="33.02"/>
-<instance part="R12" gate="G$1" x="-20.32" y="40.64" rot="R270"/>
-<instance part="GND9" gate="1" x="-20.32" y="25.4"/>
+<instance part="C1" gate="G$1" x="132.08" y="48.26"/>
+<instance part="C2" gate="G$1" x="132.08" y="33.02"/>
+<instance part="R12" gate="G$1" x="-20.32" y="43.18" rot="R270"/>
+<instance part="GND9" gate="1" x="-20.32" y="30.48"/>
 <instance part="Q3" gate="G$1" x="-10.16" y="53.34"/>
 <instance part="Q4" gate="G$1" x="0" y="53.34" rot="MR0"/>
@@
 <instance part="R16" gate="G$1" x="147.32" y="127"/>
 <instance part="R17" gate="G$1" x="147.32" y="111.76"/>
+<instance part="P-7" gate="1" x="-73.66" y="58.42"/>
+<instance part="IC2" gate="A" x="-43.18" y="99.06"/>
+<instance part="IC2" gate="B" x="160.02" y="139.7"/>
+<instance part="IC2" gate="C" x="160.02" y="124.46"/>
+<instance part="IC2" gate="D" x="160.02" y="109.22"/>
+<instance part="IC2" gate="P" x="93.98" y="38.1"/>
+<instance part="P+7" gate="1" x="93.98" y="52.832"/>
+<instance part="P-8" gate="1" x="93.98" y="24.384"/>
+<instance part="U$1" gate="G$1" x="-104.14" y="45.72"/>
 </instances>
 <busses>
@@
 <pinref part="U1" gate="G$1" pin="GND"/>
 <pinref part="GND5" gate="1" pin="GND"/>
-<wire x1="-76.2" y1="119.38" x2="-63.5" y2="119.38" width="0.1524" layer="91"/>
+<wire x1="45.72" y1="40.64" x2="58.42" y2="40.64" width="0.1524" layer="91"/>
 </segment>
 <segment>
@@
 </segment>
 <segment>
-<pinref part="CUTOFF" gate="G$1" pin="A"/>
-<pinref part="GND2" gate="1" pin="GND"/>
-<wire x1="-73.66" y1="63.5" x2="-73.66" y2="60.96" width="0.1524" layer="91"/>
-</segment>
-<segment>
 <pinref part="GND1" gate="1" pin="GND"/>
-<wire x1="55.88" y1="35.56" x2="55.88" y2="40.64" width="0.1524" layer="91"/>
-<wire x1="66.04" y1="43.18" x2="66.04" y2="40.64" width="0.1524" layer="91"/>
-<wire x1="66.04" y1="40.64" x2="66.04" y2="35.56" width="0.1524" layer="91"/>
-<wire x1="55.88" y1="40.64" x2="66.04" y2="40.64" width="0.1524" layer="91"/>
-<junction x="66.04" y="40.64"/>
+<wire x1="121.92" y1="35.56" x2="121.92" y2="40.64" width="0.1524" layer="91"/>
+<wire x1="132.08" y1="43.18" x2="132.08" y2="40.64" width="0.1524" layer="91"/>
+<wire x1="132.08" y1="40.64" x2="132.08" y2="35.56" width="0.1524" layer="91"/>
+<wire x1="121.92" y1="40.64" x2="132.08" y2="40.64" width="0.1524" layer="91"/>
+<junction x="132.08" y="40.64"/>
 <pinref part="C1" gate="G$1" pin="-"/>
 <pinref part="C2" gate="G$1" pin="+"/>
@@
 <segment>
 <pinref part="R12" gate="G$1" pin="2"/>
-<wire x1="-20.32" y1="27.94" x2="-20.32" y2="35.56" width="0.1524" layer="91"/>
+<wire x1="-20.32" y1="33.02" x2="-20.32" y2="38.1" width="0.1524" layer="91"/>
 <pinref part="GND9" gate="1" pin="GND"/>
 </segment>
@@
 <pinref part="U1" gate="G$1" pin="+12V"/>
 <pinref part="P+2" gate="1" pin="+12V"/>
-<wire x1="-76.2" y1="121.92" x2="-73.66" y2="121.92" width="0.1524" layer="91"/>
-<wire x1="-73.66" y1="121.92" x2="-73.66" y2="127" width="0.1524" layer="91"/>
+<wire x1="45.72" y1="43.18" x2="48.26" y2="43.18" width="0.1524" layer="91"/>
+<wire x1="48.26" y1="43.18" x2="48.26" y2="48.26" width="0.1524" layer="91"/>
 </segment>
 <segment>
@@
 <segment>
 <pinref part="P+1" gate="1" pin="+12V"/>
-<wire x1="66.04" y1="50.8" x2="66.04" y2="55.372" width="0.1524" layer="91"/>
+<wire x1="132.08" y1="50.8" x2="132.08" y2="55.372" width="0.1524" layer="91"/>
 <pinref part="C1" gate="G$1" pin="+"/>
 </segment>
@@
 <pinref part="U1" gate="G$1" pin="-12V"/>
 <pinref part="P-2" gate="1" pin="-12V"/>
-<wire x1="-76.2" y1="116.84" x2="-68.58" y2="116.84" width="0.1524" layer="91"/>
-<wire x1="-68.58" y1="116.84" x2="-68.58" y2="111.76" width="0.1524" layer="91"/>
+<wire x1="45.72" y1="38.1" x2="53.34" y2="38.1" width="0.1524" layer="91"/>
+<wire x1="53.34" y1="38.1" x2="53.34" y2="33.02" width="0.1524" layer="91"/>
 </segment>
 <segment>
@@
 <pinref part="IC1" gate="G$5" pin="V-"/>
 <pinref part="P-3" gate="1" pin="-12V"/>
-<wire x1="40.64" y1="16.764" x2="40.64" y2="24.13" width="0.1524" layer="91"/>
+<wire x1="106.68" y1="16.764" x2="106.68" y2="24.13" width="0.1524" layer="91"/>
 </segment>
 <segment>
 <pinref part="P-1" gate="1" pin="-12V"/>
-<wire x1="66.04" y1="27.94" x2="66.04" y2="24.384" width="0.1524" layer="91"/>
+<wire x1="132.08" y1="27.94" x2="132.08" y2="24.384" width="0.1524" layer="91"/>
 <pinref part="C2" gate="G$1" pin="-"/>
 </segment>
@@
 <pinref part="P-6" gate="1" pin="-12V"/>
 <wire x1="132.08" y1="91.44" x2="132.08" y2="93.98" width="0.1524" layer="91"/>
+</segment>
+<segment>
+<pinref part="CUTOFF" gate="G$1" pin="A"/>
+<wire x1="-73.66" y1="63.5" x2="-73.66" y2="60.96" width="0.1524" layer="91"/>
+<pinref part="P-7" gate="1" pin="-12V"/>
+</segment>
+<segment>
+<pinref part="IC2" gate="P" pin="V-"/>
+<wire x1="93.98" y1="30.48" x2="93.98" y2="26.924" width="0.1524" layer="91"/>
+<pinref part="P-8" gate="1" pin="-12V"/>
 </segment>
 </net>
@@
 <junction x="-43.18" y="17.78"/>
 <pinref part="R12" gate="G$1" pin="1"/>
-<wire x1="-20.32" y1="45.72" x2="-20.32" y2="53.34" width="0.1524" layer="91"/>
+<wire x1="-20.32" y1="48.26" x2="-20.32" y2="53.34" width="0.1524" layer="91"/>
 <junction x="-20.32" y="53.34"/>
 <pinref part="Q3" gate="G$1" pin="B"/>
@@
 <segment>
 <pinref part="U1" gate="G$1" pin="CV"/>
-<wire x1="-76.2" y1="111.76" x2="-73.66" y2="111.76" width="0.1524" layer="91"/>
-<wire x1="-73.66" y1="111.76" x2="-73.66" y2="104.14" width="0.1524" layer="91"/>
-<wire x1="-73.66" y1="104.14" x2="-91.44" y2="104.14" width="0.1524" layer="91"/>
-<wire x1="-91.44" y1="104.14" x2="-91.44" y2="45.72" width="0.1524" layer="91"/>
-<wire x1="-91.44" y1="45.72" x2="-88.9" y2="45.72" width="0.1524" layer="91"/>
+<wire x1="45.72" y1="33.02" x2="48.26" y2="33.02" width="0.1524" layer="91"/>
+<wire x1="48.26" y1="33.02" x2="48.26" y2="-17.78" width="0.1524" layer="91"/>
+<wire x1="48.26" y1="-17.78" x2="-88.9" y2="-17.78" width="0.1524" layer="91"/>
+<wire x1="-88.9" y1="-17.78" x2="-88.9" y2="45.72" width="0.1524" layer="91"/>
 <pinref part="CV1_NORM" gate="1" pin="MP"/>
 </segment>
@@
 <pinref part="IC1" gate="G$5" pin="V+"/>
 <pinref part="P+4" gate="1" pin="+12V"/>
-<wire x1="40.64" y1="57.912" x2="40.64" y2="53.34" width="0.1524" layer="91"/>
+<wire x1="106.68" y1="57.912" x2="106.68" y2="53.34" width="0.1524" layer="91"/>
+</segment>
+<segment>
+<pinref part="IC2" gate="P" pin="V+"/>
+<wire x1="93.98" y1="45.72" x2="93.98" y2="50.292" width="0.1524" layer="91"/>
+<pinref part="P+7" gate="1" pin="+12V"/>
 </segment>
 </net>
@@
 </segment>
 </net>
+<net name="N$9" class="0">
+<segment>
+<pinref part="R5" gate="G$1" pin="1"/>
+<pinref part="IC2" gate="A" pin="OUT"/>
+</segment>
+</net>
+<net name="N$11" class="0">
+<segment>
+<pinref part="R15" gate="G$1" pin="2"/>
+<pinref part="IC2" gate="B" pin="+IN"/>
+</segment>
+</net>
+<net name="N$12" class="0">
+<segment>
+<pinref part="R16" gate="G$1" pin="2"/>
+<pinref part="IC2" gate="C" pin="+IN"/>
+</segment>
+</net>
+<net name="N$13" class="0">
+<segment>
+<pinref part="R17" gate="G$1" pin="2"/>
+<pinref part="IC2" gate="D" pin="+IN"/>
+</segment>
+</net>

Commit message: parts in place
Parts:
- removed CV1, CV1_NORM, CV2: LSP10, solpad:LSP10
- removed CV2_LEVEL: 100k, pot:3RP/1610N
- removed U$1: AUDIO-JACK, erthenvar:AUDIO-JACK
- added BP_OUT, CV_1, HP_OUT, IN_1, LP_OUT: AUDIO-JACK, erthenvar:AUDIO-JACK
- added CV1_LEVEL, IN1_LEV: 100k, pot:3RP/1610N
- added Q: 50k, pot:3RP/1610N
- added R18, R19, R20, R21: 100k, rcl:R-US_0207/7
- added R22: 10k, rcl:R-US_0207/7
- added SCALE_TRIM: 10k, rcl:R-TRIMM64W
- R7: value 100k -> 10k
Connections:
- removed net N$53: R7.2
- removed net N$59: CV1.MP
- new net N$14: IC2D.-IN, IC2D.OUT, LP_OUT.TIP
- new net N$15: BP_OUT.TIP, IC2C.-IN, IC2C.OUT
- new net N$17: HP_OUT.TIP, IC2B.-IN, IC2B.OUT
- new net N$18: Q3.B, R11.1, R12.1, R6.1, R8.1
- new net N$19: Q.S, R18.2
- new net N$20: IC1B.IABC, R22.1
- new net N$21: R22.2, R7.2, SCALE_TRIM.E
- new net N$22: IN1_LEV.E, IN_1.TIP
- new net N$23: IC1G$3.OUT, R17.1, R19.2, R4.1
- new net N$24: IN1_LEV.S, R21.1
- new net N$25: Q4.C, SCALE_TRIM.A, SCALE_TRIM.S
- new net N$26: IC2A.-IN, R18.1, R19.1, R20.1, R21.2
- net GND: now also BP_OUT.RING, CV1_LEVEL.A, CV_1.RING, HP_OUT.RING, IC2A.+IN, IN1_LEV.A, IN_1.RING, LP_OUT.RING, Q.A; no longer CV2_LEVEL.A
- net N$10: now also CV1_LEVEL.S; no longer CV2_LEVEL.S
- net N$16: now also IC1A.IABC; no longer Q3.B, R11.1, R12.1, R6.1, R8.1
- net N$5: now also Q.E, R16.1
- net N$54: now also CV1_LEVEL.E, CV_1.TIP; no longer CV2.MP, CV2_LEVEL.E
- net N$55: now also CV_1.NORM; no longer CV1_NORM.MP
- net N$9: now also R15.1, R20.2
Other:
- moved on the sheet: C3, C4, CUTOFF, CUTOFF_INIT, IC1A, IC1B, IC2A, IC2B, IC2C, IC2D, Q3, Q4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
